File: radar-pcb.kicad_pcb (KiCad board)
At the start: 2 copper layers, 8 parts, among them J1 Conn_01x04_Pin, J2 Conn_01x05_Pin

Commit message: Upload
Parts:
- PIR1: value PIR Breakout JST -> Conn_01x04_Pin
- moved PIR1 0.27 mm to (31.3, 80.5)
Connections:
- ESP32-NODECMU1 pad 8: unconnected-(ESP32-NODECMU1-P33-Pad8) -> /gpio33
- PIR1 pad 4: (no net) -> /gpio33
Routing:
- net +5V: track 39.2 -> 83.8 mm, vias 0 -> 2
- net GND: track 168.5 -> 151.9 mm, vias 2 -> 6
- net /gpio33: track 0.00 -> 16.0 mm
- net /SCL: track 93.9 -> 106.0 mm, vias 0 -> 2
- net /SDA: track 87.6 -> 93.7 mm, vias 2 -> 0
- net +3.3V: track 137.2 -> 139.7 mm, vias 0 -> 3
- net /gpio39: track 54.4 -> 52.7 mm, vias 1 -> 2
- net /gpio36: track 64.0 -> 62.8 mm, vias 1 -> 2
